File: kicad/meshlight.kicad_pcb (KiCad board)
At the start: 2 copper layers, 50 x 50 mm, 59 parts, among them J1 Conn_01x05_Male, J2 Conn_01x05_Female, J3 Barrel_Jack_Switch, Q1 BC847, Q2 BC847, Q3 BC847, Q4 BC847, Q5 BC847, Q6 BC847, Q7 BC847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

Commit message: basic rough placing of all components
Parts:
- J1, J2, J3, U2: moved to B.Cu
- moved U2 193.6 mm to (213.4, 43.8), turned to 180 degrees
- moved C1 191.6 mm to (213.0, 56.5), turned to 180 degrees
- moved C2 189.1 mm to (213.1, 59.1)
- moved J3 185.0 mm to (201.9, 32.4), turned to 180 degrees
- moved R6 183.5 mm to (217.2, 43.8), turned to 180 degrees
- moved U1 169.2 mm to (206.4, 59.1), turned to 180 degrees
- moved C3 166.5 mm to (196.2, 36.2), turned to 270 degrees
- moved R1 137.8 mm to (207.0, 48.9)
- moved R11 130.9 mm to (207.0, 46.4)
- moved J1 124.2 mm to (181.0, 92.1)
- moved D3 122.8 mm to (160.0, 78.7), turned to 270 degrees
- moved Q7 116.2 mm to (170.8, 88.3), turned to 180 degrees
- moved Q1 114.2 mm to (131.7, 67.9)
- moved R13 112.2 mm to (174.6, 87.0)
- moved Q3 111.1 mm to (168.3, 99.7), turned to 180 degrees
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
Commit message: routed pcb
Parts:
- added G***: LOGO, kicad:laborlogo, F.Cu at (150.2, 87.0)
- added H1: MountingHole, MountingHole:MountingHole_4.3mm_M4, F.Cu at (123.8, 62.9)
- added H2: MountingHole, MountingHole:MountingHole_4.3mm_M4, F.Cu at (176.5, 62.9)
- added H3: MountingHole_Pad, MountingHole:MountingHole_4.3mm_M4, F.Cu at (176.5, 111.1)
- added H4: MountingHole, MountingHole:MountingHole_4.3mm_M4, F.Cu at (123.8, 111.1)
- moved R6 98.5 mm to (144.1, 109.9), turned to 270 degrees
- moved R1 93.9 mm to (135.6, 109.9), turned to 270 degrees
- moved C3 80.3 mm to (165.7, 110.5), turned to 0 degrees
- moved J3 77.6 mm to (170.8, 103.5)
- moved R11 52.6 mm to (157.5, 64.1), turned to 270 degrees
- moved R12 52.5 mm to (155.4, 64.1), turned to 90 degrees
- moved C1 52.2 mm to (161.3, 64.1), turned to 90 degrees
- moved D9 47.9 mm to (152.4, 64.1), turned to 90 degrees
- moved U2 44.7 mm to (176.5, 69.2)
- moved C2 42.3 mm to (171.6, 67.1), turned to 90 degrees
- moved R7 41.4 mm to (142.2, 109.9), turned to 90 degrees
- moved U1 40.1 mm to (167.0, 66.7), turned to 270 degrees
- moved D8 35.7 mm to (139.1, 109.9)
- moved R2 33.0 mm to (133.9, 109.9), turned to 90 degrees
- moved D7 27.0 mm to (130.8, 109.9)
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Routing:
- net Net-(D8-Pad1): track 0.00 -> 133.5 mm
- net +3V3: track 0.00 -> 130.1 mm, vias 0 -> 5
- net /LED_G: track 0.00 -> 114.4 mm, vias 0 -> 1
- net Net-(D7-Pad1): track 0.00 -> 109.4 mm, vias 0 -> 2
- net /LED_R: track 0.00 -> 102.7 mm, vias 0 -> 1
- net /LED_B: track 0.00 -> 93.5 mm, vias 0 -> 1
- net Net-(DB3-Pad1): track 0.00 -> 91.8 mm
- net Net-(D9-Pad1): track 0.00 -> 78.3 mm, vias 0 -> 2
- net Net-(DG3-Pad1): track 0.00 -> 65.9 mm
- net GND: track 0.00 -> 58.8 mm, vias 0 -> 19
- net /LR1: track 0.00 -> 57.4 mm, vias 0 -> 1
- net Net-(DR3-Pad1): track 0.00 -> 55.2 mm
- net /LR3: track 0.00 -> 55.0 mm
- net /LR2: track 0.00 -> 53.9 mm, vias 0 -> 2
- net /LB3: track 0.00 -> 46.2 mm
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- added copper zone on B.Cu, net GND
Other:
- board size 50 x 50 mm -> 60.3 x 55.9 mm
- net class Default: trace_width 0.25 -> 0.3048
- net class Power added: clearance 0.26, trace_width 0.6096, via_dia 1, via_drill 0.5
- board text added: "+ R G B -"
- board text added: "EXT OUT"
- board text added: "ID:"
- board text added: "IN"
- board text added: "meshlight v1.0 by e7p"

Commit message: added gerber files for fab
Other:
- board text added: "JLCJLCJLCJLC"
Changed lines of the file:
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@@
   (general
     (thickness 1.6)
-    (drawings 23)
+    (drawings 20)
     (tracks 739)
     (zones 0)
@@
   (layers
     (0 F.Cu signal)
-    (31 B.Cu signal hide)
+    (31 B.Cu signal)
     (32 B.Adhes user hide)
-    (33 F.Adhes user)
+    (33 F.Adhes user hide)
     (34 B.Paste user hide)
-    (35 F.Paste user)
-    (36 B.SilkS user hide)
+    (35 F.Paste user hide)
+    (36 B.SilkS user)
     (37 F.SilkS user)
-    (38 B.Mask user hide)
-    (39 F.Mask user hide)
+    (38 B.Mask user)
+    (39 F.Mask user)
     (40 Dwgs.User user hide)
     (41 Cmts.User user hide)
@@
     (visible_elements FFFFFF7F)
     (pcbplotparams
-      (layerselection 0x010fc_ffffffff)
+      (layerselection 0x010f0_ffffffff)
       (usegerberextensions false)
       (usegerberattributes false)
@@
       (outputformat 1)
       (mirror false)
-      (drillshape 1)
+      (drillshape 0)
       (scaleselection 1)
-      (outputdirectory ""))
+      (outputdirectory "gerber/"))
   )
   (net 0 "")
@@
       (net 2 GND))
   )
+  (gr_text JLCJLCJLCJLC (at 166.0525 113.665) (layer B.SilkS)
+    (effects (font (size 1 1) (thickness 0.15)) (justify mirror))
+  )
   (gr_text "+  R  G  B  -" (at 173.99 86.995 270) (layer B.SilkS)
     (effects (font (size 1 1) (thickness 0.15)) (justify mirror))
@@
   (gr_arc (start 123.825 111.125) (end 120.015 111.125) (angle -90) (layer Edge.Cuts) (width 0.05))
   (gr_arc (start 123.825 62.865) (end 123.825 59.055) (angle -90) (layer Edge.Cuts) (width 0.05))
-  (target plus (at 123.825 62.865) (size 5) (width 0.05) (layer Edge.Cuts))
-  (target plus (at 123.825 111.125) (size 5) (width 0.05) (layer Edge.Cuts))
-  (target plus (at 176.53 111.125) (size 5) (width 0.05) (layer Edge.Cuts))
-  (target plus (at 176.53 62.865) (size 5) (width 0.05) (layer Edge.Cuts))
   (gr_line (start 120.015 62.865) (end 120.015 111.125) (layer Edge.Cuts) (width 0.05))
   (gr_line (start 176.53 114.935) (end 123.825 114.935) (layer Edge.Cuts) (width 0.05))
